File: atmo_sense/atmo_sense.kicad_pcb (KiCad board)
At the start: 4 copper layers, 90 x 60 mm, 54 parts, among them J1 Conn_01x04_Pin, J2 USB-C, J3 TB007-508-02BE, J4 Conn_02x05_Top_Bottom, SW1 SW_Push, SW2 SW_Push, SW3 SW_Push, SW4 SW_Push, U1 USBLC6-2SC6, U2 ESP32-C3FH4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

Commit message: Backup
Parts:
- removed SW4: SW_Push, Button_Switch_SMD:SW_SPST_PTS810
- added J5: Conn_01x04_Pin, Connector_PinSocket_2.00mm:PinSocket_2x02_P2.00mm_Vertical_SMD, F.Cu at (131.5, 57.1)
- moved C9 97.7 mm to (123.2, 65.5), turned to -90 degrees
- moved C10 90.6 mm to (116.9, 67.1), turned to -90 degrees
- moved C2 86.4 mm to (121.8, 65.5), turned to -90 degrees
- moved C1 81.4 mm to (114.8, 57.7), turned to 180 degrees
- moved C4 80.0 mm to (114.8, 58.8), turned to 180 degrees
- moved C3 76.6 mm to (108.6, 61.4), turned to -90 degrees
- moved C5 74.3 mm to (110.4, 62.4)
- moved C8 71.6 mm to (128.0, 61.2), turned to -90 degrees
- moved L1 70.2 mm to (110.4, 61.4)
- moved D1 69.9 mm to (105.6, 75.8), turned to 90 degrees
- moved C11 68.2 mm to (112.0, 62.0), turned to -90 degrees
- moved R6 64.4 mm to (135.1, 53.6)
- moved C7 48.0 mm to (121.5, 57.6)
- moved SW3 43.7 mm to (123.9, 55.0), turned to -90 degrees
- moved J4 41.9 mm to (135.6, 80.5), turned to -90 degrees
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Connections:
- C1 pad 1: +3V3 -> +3.3V
- C10 pad 1: +3V3 -> +3.3V
- C2 pad 1: +3V3 -> +3.3V
- C3 pad 1: +3V3 -> +3.3V
- C4 pad 1: +3V3 -> +3.3V
- C5 pad 1: +3V3 -> +3.3V
- C9 pad 1: +3V3 -> +3.3V
- D1 pad 2: +3V3 -> +3.3V
- L1 pad 1: +3V3 -> +3.3V
- U2 pad 11: +3V3 -> +3.3V
- U2 pad 17: +3V3 -> +3.3V
- U2 pad 18: +3V3 -> +3.3V
- U2 pad 31: +3V3 -> +3.3V
- U2 pad 32: +3V3 -> +3.3V
Routing:
- net +3.3V: track 0.00 -> 132.7 mm, vias 0 -> 5
- net +5V: track 0.00 -> 87.7 mm, vias 0 -> 5
- net Net-(J3-Pin_2): track 0.00 -> 36.8 mm
- net /RX_PMS: track 0.00 -> 34.1 mm, vias 0 -> 2
- net /CHIP_EN: track 0.00 -> 32.8 mm
- net /TX_PMS: track 0.00 -> 30.3 mm, vias 0 -> 2
- net /USB_DP: track 0.00 -> 26.9 mm
- net /SDA: track 0.00 -> 26.4 mm, vias 0 -> 2
- net /USB_DN: track 0.00 -> 25.5 mm
- net /SCL: track 0.00 -> 23.7 mm, vias 0 -> 2
- net /SEL_SW: track 0.00 -> 23.2 mm, vias 0 -> 2
- net Net-(J3-Pin_1): track 0.00 -> 18.2 mm
- net Net-(PS1-AC/L): track 0.00 -> 14.2 mm
- net /CFG_SW: track 0.00 -> 12.0 mm
- net /GPI09: track 0.00 -> 11.3 mm
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Other:
- board size 90 x 60 mm -> 57 x 59 mm
- board text added: "ATMOSENSE V1.0"
- board text added: "BOOT"
- board text added: "CONFIG"
- board text added: "RESET"
- board text added: "SELECT"

Commit message: PCB design
Parts:
- added H1: MountingHole, MountingHole:MountingHole_2mm, F.Cu at (140.4, 56.3)
- added H2: MountingHole, MountingHole:MountingHole_2mm, F.Cu at (145.9, 106.4)
- added H3: MountingHole, MountingHole:MountingHole_2mm, F.Cu at (99.1, 90.0)
- J1: renamed from J5; footprint Connector_PinSocket_2.00mm:PinSocket_2x02_P2.00mm_Vertical_SMD -> Connector_PinSocket_2.00mm:PinSocket_2x02_P2.00mm_Vertical
- U4: value LM1117LD-3.3 -> AMS1117-3.3; footprint Package_SON:WSON-8-1EP_4x4mm_P0.8mm_EP2.2x3mm -> Package_TO_SOT_SMD:SOT-223-3_TabPin2
- moved RV1 7.91 mm to (150.5, 98.0), turned to 180 degrees
- moved C22 7.83 mm to (109.2, 77.5), turned to 90 degrees
- moved F1 7.03 mm to (151.9, 102.8)
- moved D1 5.04 mm to (109.2, 79.3)
- moved C19 4.81 mm to (111.6, 80.0), turned to -90 degrees
- moved U3 4.58 mm to (112.8, 77.1)
- moved C20 4.55 mm to (113.7, 79.5)
- moved R9 2.35 mm to (144.7, 57.2)
- moved U1 2.35 mm to (143.3, 61.3)
- moved J3 2.35 mm to (151.9, 60.7)
- moved C21 2.27 mm to (101.0, 84.8), turned to -90 degrees
- moved J2 2.19 mm to (116.7, 80.5)
- moved J1 2.03 mm to (133.5, 57.0)
- moved U4 1.97 mm to (104.1, 78.9), turned to 0 degrees
- moved R6 1.73 mm to (128.1, 55.0)
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- renumbered J1 to J2, J2 to J3, J3 to J4, J4 to J5, R6 to R5, R5 to R6
Connections:
- net /CHIP_EN renamed /RESET
- U4 pad 2: +5V -> +3.3V
Routing:
- net Net-(J4-Pin_2): track 36.8 -> 24.7 mm
- net +3.3V: track 132.7 -> 144.7 mm, vias 5 -> 6
- net /CC1: track 4.66 -> 11.5 mm
- net /RF_ANT: track 1.03 -> 7.11 mm
- net Net-(J1-Pin_1): track 10.6 -> 5.55 mm
- net /SDA: track 26.4 -> 22.8 mm
- net Net-(J4-Pin_1): track 18.2 -> 14.8 mm
- net /LNA_IN: track 1.03 -> 4.32 mm
- net /SCL: track 23.7 -> 20.7 mm
- net Net-(PS1-AC/L): track 14.2 -> 17.1 mm
- net Net-(C15-Pad1): track 2.53 -> 4.30 mm
- net /USB_DP: track 26.9 -> 28.6 mm
- net /USB_DN: track 25.5 -> 27.2 mm
- net /XTAL_32_N: track 9.81 -> 8.13 mm
- net /GPI09: track 11.3 -> 12.8 mm
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- added copper zone on B.Cu, net GND
- added copper zone on F.Cu, net GND
- added copper zone on In1.Cu, net GND
- added copper zone on In2.Cu, net GND
Other:
- board size 57 x 59 mm -> 60 x 58 mm
- board text added: "DANGER!"

Commit message: PCB
Parts:
- F1: footprint SamacSys_Parts:FUSC6125X236N -> Fuse:Fuse_2512_6332Metric
Routing:
- net Net-(PS1-AC/L): track 17.1 -> 17.8 mm
