File: atmo_sense/atmo_sense.kicad_sch (KiCad schematic)
At the start: 54 parts, among them J1 Conn_01x04_Pin, J2 USB-C, J3 TB007-508-02BE, J4 Conn_02x05_Top_Bottom, SW1 SW_Push, SW2 SW_Push, SW3 SW_Push, SW4 SW_Push, U1 USBLC6-2SC6, U2 ESP32-C3FH4, U3 BME680, U4 LM1117LD-3.3, Y1 ECS-400-10-36B2-CKM-TR, Y2 Crystal

Commit message: Backup
Parts:
- removed SW4: SW_Push, Button_Switch_SMD:SW_SPST_PTS810, symbol Switch:SW_Push
- added J5: Conn_01x04_Pin, Connector_PinSocket_2.00mm:PinSocket_2x02_P2.00mm_Vertical_SMD, symbol Connector:Conn_01x04_Pin
Connections:
- net +3V3 is gone; now on net +3.3V: C1.1, C10.1, C2.1, C3.1, C4.1, C5.1, C9.1, D1.2 (A2), L1.1, U2.11 (VDD3P3_RTC), U2.17 (VDD3P3_CPU), U2.18 (VDD_SPI), U2.31 (VDDA), U2.32 (VDDA)
- net SEL_SW: now also J5.3 (Pin_3), J5.4 (Pin_4)
- net at R6.1: now also J5.1 (Pin_1), J5.2 (Pin_2)
Other:
- moved on the sheet: C8, R6

Commit message: PCB design
Parts:
- removed U4: LM1117LD-3.3, Package_SON:WSON-8-1EP_4x4mm_P0.8mm_EP2.2x3mm, symbol Regulator_Linear:LM1117LD-3.3
- added H1, H2, H3: MountingHole, MountingHole:MountingHole_2mm, symbol Mechanical:MountingHole
- added U4: AMS1117-3.3, Package_TO_SOT_SMD:SOT-223-3_TabPin2, symbol Regulator_Linear:AMS1117-3.3
- C12, C13, L2: now fitted
- F1: footprint SamacSys_Parts:FUSC6125X236N -> Fuse:Fuse_2512_6332Metric
- J1: renamed from J5; footprint Connector_PinSocket_2.00mm:PinSocket_2x02_P2.00mm_Vertical_SMD -> Connector_PinSocket_2.00mm:PinSocket_2x02_P2.00mm_Vertical
- renumbered J1 to J2, J2 to J3, J3 to J4, J4 to J5, R6 to R5, R5 to R6
Connections:
- net +3.3V: now also U4.2 (VO)
- net +5V: now also U4.3 (VI)
- net GND: now also U4.1 (GND)
- net CHIP_EN renamed RESET

Commit message: PCB
Other:
- note added: "FUROS PARA FIXAÇÃO"
- moved on the sheet: H1, H2, H3
Changed lines of the file:
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@@
 		)
 	)
+	(text "FUROS PARA FIXAÇÃO"
+		(exclude_from_sim no)
+		(at 101.6 191.516 0)
+		(effects
+			(font
+				(size 1.27 1.27)
+			)
+		)
+	)
 	(text "BOOT MODE"
 		(exclude_from_sim no)
@@
 		)
 	)
+	(polyline
+		(pts
+			(xy 91.44 189.23) (xy 210.82 189.23)
+		)
+		(stroke
+			(width 0)
+			(type dash)
+		)
+	)
 	(wire
 		(pts
@@
 	(symbol
 		(lib_id "Mechanical:MountingHole")
-		(at 111.76 227.33 0)
+		(at 151.13 198.12 0)
 		(unit 1)
 		(exclude_from_sim no)
@@
 		(fields_autoplaced yes)
 		(property "Reference" "H3"
-			(at 114.3 226.0599 0)
+			(at 153.67 196.8499 0)
 			(effects
 				(font
@@
 		)
 		(property "Value" "MountingHole"
-			(at 114.3 228.5999 0)
+			(at 153.67 199.3899 0)
 			(effects
 				(font
@@
 		)
 		(property "Footprint" "MountingHole:MountingHole_2mm"
-			(at 111.76 227.33 0)
+			(at 151.13 198.12 0)
 			(effects
 				(font
@@
 		)
 		(property "Datasheet" "~"
-			(at 111.76 227.33 0)
+			(at 151.13 198.12 0)
 			(effects
 				(font
@@
 		)
 		(property "Description" ""
-			(at 111.76 227.33 0)
+			(at 151.13 198.12 0)
 			(effects
 				(font
@@
 	(symbol
 		(lib_id "Mechanical:MountingHole")
-		(at 111.76 212.09 0)
+		(at 102.87 198.12 0)
 		(unit 1)
 		(exclude_from_sim no)
@@
 		(fields_autoplaced yes)
 		(property "Reference" "H1"
-			(at 114.3 210.8199 0)
+			(at 105.41 196.8499 0)
 			(effects
 				(font
@@
 		)
 		(property "Value" "MountingHole"
-			(at 114.3 213.3599 0)
+			(at 105.41 199.3899 0)
 			(effects
 				(font
@@
 		)
 		(property "Footprint" "MountingHole:MountingHole_2mm"
-			(at 111.76 212.09 0)
+			(at 102.87 198.12 0)
 			(effects
 				(font
@@
 		)
 		(property "Datasheet" "~"
-			(at 111.76 212.09 0)
+			(at 102.87 198.12 0)
 			(effects
 				(font
@@
 		)
 		(property "Description" ""
-			(at 111.76 212.09 0)
+			(at 102.87 198.12 0)
 			(effects
 				(font
@@
 	(symbol
 		(lib_id "Mechanical:MountingHole")
-		(at 111.76 219.71 0)
+		(at 127 198.12 0)
 		(unit 1)
 		(exclude_from_sim no)
@@
 		(fields_autoplaced yes)
 		(property "Reference" "H2"
-			(at 114.3 218.4399 0)
+			(at 129.54 196.8499 0)
 			(effects
 				(font
@@
 		)
 		(property "Value" "MountingHole"
-			(at 114.3 220.9799 0)
+			(at 129.54 199.3899 0)
 			(effects
 				(font
@@
 		)
 		(property "Footprint" "MountingHole:MountingHole_2mm"
-			(at 111.76 219.71 0)
+			(at 127 198.12 0)
 			(effects
 				(font
@@
 		)
 		(property "Datasheet" "~"
-			(at 111.76 219.71 0)
+			(at 127 198.12 0)
 			(effects
 				(font
@@
 		)
 		(property "Description" ""
-			(at 111.76 219.71 0)
+			(at 127 198.12 0)
 			(effects
 				(font
